File: KiCad/Robot_Electronic_Design/Robot_Electronic_Design.kicad_pcb (KiCad board)
At the start: 2 copper layers, 3 parts, among them J1 Conn_01x19_Female, J2 Conn_01x19_Female, U1 L298N

Commit message: Update Kicad Files
Parts:
- removed J1, J2: Conn_01x19_Female, Connector_PinSocket_2.54mm:PinSocket_1x19_P2.54mm_Vertical
- added U2: NEO-6M, NEO-6M:NEO-6M, F.Cu at (166.3, 43.0)
- added U3: HC-SR04, HC-SR04:XCVR_HC-SR04, F.Cu at (103.9, 18.1)
- added U4: HC-SR04, HC-SR04:XCVR_HC-SR04, F.Cu at (103.9, 39.9)
- added U5: HC-SR04, HC-SR04:XCVR_HC-SR04, F.Cu at (103.9, 61.7)
- added U6: L298N, Package_TO_SOT_THT:TO-220-15_P2.54x2.54mm_StaggerOdd_Lead4.58mm_Vertical, F.Cu at (155.6, 29.1)
- U1: value L298N -> ESP32-DEVKITC-32D; footprint Package_TO_SOT_THT:TO-220-15_P2.54x2.54mm_StaggerOdd_Lead4.58mm_Vertical -> esp32:MODULE_ESP32-DEVKITC-32D
- moved U1 83.5 mm to (43.4, 47.0)

Commit message: test: DC Motors
Parts:
- added C1: 10uF, Capacitor_THT:CP_Radial_D5.0mm_P2.00mm, F.Cu at (198.8, 30.3)
- added C2: 10uF, Capacitor_THT:CP_Radial_D5.0mm_P2.00mm, F.Cu at (198.8, 36.9)
- added J1: Conn_01x19_Female, Connector_PinSocket_2.54mm:PinSocket_1x19_P2.54mm_Vertical, F.Cu at (189.6, 29.4)
- added J2: Conn_01x19_Female, Connector_PinSocket_2.54mm:PinSocket_1x19_P2.54mm_Vertical, F.Cu at (194.2, 29.4)
- added M1: Motor_DC, Connector_PinHeader_2.00mm:PinHeader_2x01_P2.00mm_Vertical, F.Cu at (198.5, 42.2)
- added M2: Motor_DC, Connector_PinHeader_2.00mm:PinHeader_2x01_P2.00mm_Vertical, F.Cu at (198.5, 46.2)
- added M3: Water Pump, Connector_PinHeader_2.00mm:PinHeader_2x01_P2.00mm_Vertical, F.Cu at (198.5, 50.3)
- added U9: AMS1117-5.0, Package_TO_SOT_SMD:SOT-223-3_TabPin2, F.Cu at (201.4, 56.5)
- renumbered U5 to U3, U3 to U5
Connections:
- U3 pad 1: unconnected-(U5-VCC-Pad1) -> Vin
- U3 pad 2: unconnected-(U5-TRIG-Pad2) -> /TRIG_1
- U3 pad 3: unconnected-(U5-ECHO-Pad3) -> /ECHO_1
- U3 pad 4: unconnected-(U5-GND-Pad4) -> GND
- U4 pad 1: unconnected-(U4-VCC-Pad1) -> Vin
- U4 pad 2: unconnected-(U4-TRIG-Pad2) -> /TRIG_2
- U4 pad 3: unconnected-(U4-ECHO-Pad3) -> /ECHO_2
- U4 pad 4: unconnected-(U4-GND-Pad4) -> GND
- U5 pad 1: unconnected-(U3-VCC-Pad1) -> Vin
- U5 pad 2: unconnected-(U3-TRIG-Pad2) -> /TRIG_3
- U5 pad 3: unconnected-(U3-ECHO-Pad3) -> /ECHO_3
- U5 pad 4: unconnected-(U3-GND-Pad4) -> GND
- U6 pad 10: unconnected-(U6-IN3-Pad10) -> /IN3
- U6 pad 11: unconnected-(U6-EnB-Pad11) -> /ENB
- U6 pad 12: unconnected-(U6-IN4-Pad12) -> /IN4
- U6 pad 13: unconnected-(U6-OUT3-Pad13) -> /MOTOR_2_OUT1
- U6 pad 14: unconnected-(U6-OUT4-Pad14) -> /MOTOR_2_OUT2
- U6 pad 2: unconnected-(U6-OUT1-Pad2) -> /MOTOR_1_OUT1
- U6 pad 3: unconnected-(U6-OUT2-Pad3) -> /MOTOR_1_OUT2
- U6 pad 4: unconnected-(U6-Vs-Pad4) -> VCC
- U6 pad 5: unconnected-(U6-IN1-Pad5) -> /IN1
- U6 pad 6: unconnected-(U6-EnA-Pad6) -> /ENA
- U6 pad 7: unconnected-(U6-IN2-Pad7) -> /IN2
- U6 pad 8: unconnected-(U6-GND-Pad8) -> GND
- U6 pad 9: unconnected-(U6-Vss-Pad9) -> Vin
